Commit message: descriptio

File: ar_description/urdf/ar.ros2_control.xacro (robot description, xacro)
@@ -18,6 +18,6 @@
       <joint name="joint_1">
         <command_interface name="position">
-          <param name="min">{-170*pi/180}</param>
-          <param name="max">{170*pi/180}</param>
+          <param name="min">{-184*pi/180}</param>
+          <param name="max">{150*pi/180}</param>
         </command_interface>
         <state_interface name="position">
@@ -28,5 +28,5 @@
       <joint name="joint_2">
         <command_interface name="position">
-          <param name="min">{-42*pi/180}</param>
+          <param name="min">{-47*pi/180}</param>
           <param name="max">{90*pi/180}</param>
         </command_interface>
@@ -38,6 +38,6 @@
       <joint name="joint_3">
         <command_interface name="position">
-          <param name="min">{-89*pi/180}</param>
-          <param name="max">{52*pi/180}</param>
+          <param name="min">{-90*pi/180}</param>
+          <param name="max">{62*pi/180}</param>
         </command_interface>
         <state_interface name="position">
@@ -48,6 +48,6 @@
       <joint name="joint_4">
         <command_interface name="position">
-          <param name="min">{-165*pi/180}</param>
-          <param name="max">{165*pi/180}</param>
+          <param name="min">{-161*pi/180}</param>
+          <param name="max">{169*pi/180}</param>
         </command_interface>
         <state_interface name="position">
@@ -58,6 +58,6 @@
       <joint name="joint_5">
         <command_interface name="position">
-          <param name="min">{-105*pi/180}</param>
-          <param name="max">{105*pi/180}</param>
+          <param name="min">{-100*pi/180}</param>
+          <param name="max">{100*pi/180}</param>
         </command_interface>
         <state_interface name="position">
@@ -68,6 +68,6 @@
       <joint name="joint_6">
         <command_interface name="position">
-          <param name="min">{-155*pi/180}</param>
-          <param name="max">{155*pi/180}</param>
+          <param name="min">{-170*pi/180}</param>
+          <param name="max">{150*pi/180}</param>
         </command_interface>
         <state_interface name="position">

File: ar_description/urdf/ar.urdf.xacro (robot description, xacro)
@@ -1,5 +1,5 @@
 <?xml version="1.0"?>
 <robot xmlns:xacro="http://wiki.ros.org/xacro" name="$(arg ar_model)">
-  <xacro:arg name="include_gripper" default="true"/>
+  <xacro:arg name="include_gripper" default="false"/>
   <xacro:include filename="$(find ar_description)/urdf/ar_macro.xacro"/>
   <link name="world" />

File: ar_description/urdf/ar_macro.xacro (robot description, xacro)
@@ -19,5 +19,5 @@
       </inertial>
       <visual>
-        <origin rpy="0 0 0" xyz="0 0 0"/>
+        <origin rpy="${pi/2} 0 0" xyz="0 0 0"/>
         <geometry>
           <mesh filename="file://$(find ar_description)/meshes/${robot_parameters['mesh_dir']}/base_link.STL"/>
@@ -28,5 +28,5 @@
       </visual>
       <collision>
-        <origin rpy="0 0 0" xyz="0 0 0"/>
+        <origin rpy="${pi/2} 0 0" xyz="0 0 0"/>
         <geometry>
           <mesh filename="file://$(find ar_description)/meshes/${robot_parameters['mesh_dir']}/base_link.STL"/>
@@ -57,9 +57,9 @@
     </link>
     <joint name="joint_1" type="revolute">
-      <origin rpy="${pi} 0 0" xyz="0 0 0"/>
+      <origin rpy="${pi/2} 0 0" xyz="0 0 0"/>
       <parent link="base_link"/>
       <child link="link_1"/>
-      <axis xyz="0 0 1"/>
-      <limit lower="${-170.0 / 180.0 * pi}" upper="${170.0 / 180.0 * pi}" effort="0" velocity="0.5"/>
+      <axis xyz="0 -1 0"/>
+      <limit lower="${-184.0 / 180.0 * pi}" upper="${150.0 / 180.0 * pi}" effort="0" velocity="0.5"/>
     </joint>
     <link name="link_2">
@@ -86,9 +86,9 @@
     </link>
     <joint name="joint_2" type="revolute">
-      <origin rpy="1.5708 0 -1.5708" xyz="0 0.0642 -0.16977"/>
+      <origin rpy="0 0 0" xyz="0.06384 0.1736 0"/>
       <parent link="link_1"/>
       <child link="link_2"/>
       <axis xyz="0 0 -1"/>
-      <limit lower="${-42.0 / 180.0 * pi}" upper="${90.0 / 180.0 * pi}" effort="0.5" velocity="0.5"/>
+      <limit lower="${-47.0 / 180.0 * pi}" upper="${90.0 / 180.0 * pi}" effort="0.5" velocity="0.5"/>
     </joint>
     <link name="link_3">
@@ -115,9 +115,9 @@
     </link>
     <joint name="joint_3" type="revolute">
-      <origin rpy="0 0 3.1416" xyz="0 -0.305 0.007"/>
+      <origin rpy="0 0 0" xyz="0 0.34997 0.0046"/>
       <parent link="link_2"/>
       <child link="link_3"/>
       <axis xyz="0 0 -1"/>
-      <limit lower="${-89.0 / 180.0 * pi}" upper="${52.0 / 180.0 * pi}" effort="0" velocity="0.5"/>
+      <limit lower="${-90.0 / 180.0 * pi}" upper="${62.0 / 180.0 * pi}" effort="0" velocity="0.5"/>
     </joint>
     <link name="link_4">
@@ -144,9 +144,9 @@
     </link>
     <joint name="joint_4" type="revolute">
-      <origin rpy="1.5708 0 -1.5708" xyz="0 0 0.0"/>
+      <origin rpy="0 0 0" xyz="0 0 0.0"/>
       <parent link="link_3"/>
       <child link="link_4"/>
-      <axis xyz="0 0 -1"/>
-      <limit lower="${-1 * robot_parameters['j4_limit']}" upper="${robot_parameters['j4_limit']}" effort="0" velocity="0.5"/>
+      <axis xyz="1 0 0"/>
+      <limit lower="${-161.0 / 180.0 * pi}" upper="${169.0 / 180.0 * pi}" effort="0" velocity="0.5"/>
     </joint>
     <link name="link_5">
@@ -173,9 +173,9 @@
     </link>
     <joint name="joint_5" type="revolute">
-      <origin rpy="${pi} 0 -1.5708" xyz="0 0 -0.22263"/>
+      <origin rpy="0 0 0" xyz="0.27435 0 0"/>
       <parent link="link_4"/>
       <child link="link_5"/>
-      <axis xyz="1 0 0"/>
-      <limit lower="${-105.0 / 180.0 * pi}" upper="${105.0 / 180.0 * pi}" effort="0" velocity="1.0"/>
+      <axis xyz="0 0 -1"/>
+      <limit lower="${-100.0 / 180.0 * pi}" upper="${100.0 / 180.0 * pi}" effort="0" velocity="1.0"/>
     </joint>
     <link name="link_6">
@@ -202,9 +202,9 @@
     </link>
     <joint name="joint_6" type="revolute">
-      <origin rpy="0 0 3.1416" xyz="0.000 0 ${robot_parameters['l6_length']}"/>
+      <origin rpy="0 0 0" xyz="0.0384 0 0"/>
       <parent link="link_5"/>
       <child link="link_6"/>
-      <axis xyz="0 0 1"/>
-      <limit lower="${-1.0 * robot_parameters['j6_limit']}" upper="${robot_parameters['j6_limit']}" effort="0" velocity="1.0"/>
+      <axis xyz="1 0 0"/>
+      <limit lower="${-170.0 / 180.0 * pi}" upper="${150.0 / 180.0 * pi}" effort="0" velocity="1.0"/>
     </joint>
     <!-- center of the end effector mounting surface on link_6 -->
