Commit message: urdf modifications

File: src/ar_description/urdf/ar.urdf.xacro (robot description, xacro)
@@ -1,11 +1,11 @@
 <?xml version="1.0"?>
 <robot xmlns:xacro="http://wiki.ros.org/xacro" name="$(arg ar_model)">
-  <xacro:arg name="include_gripper" default="false"/>
+  <xacro:arg name="include_gripper" default="False"/>
   <xacro:include filename="$(find ar_description)/urdf/ar_macro.xacro"/>
   <link name="world" />
   <xacro:ar_robot
     parent="world"
-    robot_parameters_file="$(find ar_description)/config/$(arg ar_model).yaml"
   >
+    <!-- robot_parameters_file="$(find ar_description)/config/$(arg ar_model).yaml" -->
     <origin xyz="0 0 0" rpy="0 0 0" />
   </xacro:ar_robot>

File: src/ar_description/urdf/ar_macro.xacro (robot description, xacro)
@@ -4,7 +4,7 @@
     parent
     *origin
-    robot_parameters_file
   ">
-    <xacro:property name="robot_parameters" value="${xacro.load_yaml(robot_parameters_file)}"/>
+    <!-- robot_parameters_file -->
+    <!-- <xacro:property name="robot_parameters" value="${xacro.load_yaml(robot_parameters_file)}"/> -->
     <joint name="base_joint" type="fixed">
       <xacro:insert_block name="origin" />
@@ -21,5 +21,5 @@
         <origin rpy="${pi/2} 0 0" xyz="0 0 0"/>
         <geometry>
-          <mesh filename="file://$(find ar_description)/meshes/${robot_parameters['mesh_dir']}/base_link.STL"/>
+          <mesh filename="file://$(find ar_description)/meshes/ar4/base_link.STL"/>
         </geometry>
         <material name="">
@@ -30,5 +30,5 @@
         <origin rpy="${pi/2} 0 0" xyz="0 0 0"/>
         <geometry>
-          <mesh filename="file://$(find ar_description)/meshes/${robot_parameters['mesh_dir']}/base_link.STL"/>
+          <mesh filename="file://$(find ar_description)/meshes/ar4/base_link.STL"/>
         </geometry>
       </collision>
@@ -43,14 +43,14 @@
         <origin rpy="0 0 0" xyz="0 0 0"/>
         <geometry>
-          <mesh filename="file://$(find ar_description)/meshes/${robot_parameters['mesh_dir']}/link_1.STL"/>
-        </geometry>
-        <material name="">
-          <color rgba="1 1 0 1"/>
-        </material>
-      </visual>
-      <collision>
-        <origin rpy="0 0 0" xyz="0 0 0"/>
-        <geometry>
-          <mesh filename="file://$(find ar_description)/meshes/${robot_parameters['mesh_dir']}/link_1.STL"/>
+          <mesh filename="file://$(find ar_description)/meshes/ar4/link_1.STL"/>
+        </geometry>
+        <material name="">
+          <color rgba="1 1 0 1"/>
+        </material>
+      </visual>
+      <collision>
+        <origin rpy="0 0 0" xyz="0 0 0"/>
+        <geometry>
+          <mesh filename="file://$(find ar_description)/meshes/ar4/link_1.STL"/>
         </geometry>
       </collision>
@@ -72,14 +72,14 @@
         <origin rpy="0 0 0" xyz="0 0 0"/>
         <geometry>
-          <mesh filename="file://$(find ar_description)/meshes/${robot_parameters['mesh_dir']}/link_2.STL"/>
-        </geometry>
-        <material name="">
-          <color rgba="1 1 0 1"/>
-        </material>
-      </visual>
-      <collision>
-        <origin rpy="0 0 0" xyz="0 0 0"/>
-        <geometry>
-          <mesh filename="file://$(find ar_description)/meshes/${robot_parameters['mesh_dir']}/link_2.STL"/>
+          <mesh filename="file://$(find ar_description)/meshes/ar4/link_2.STL"/>
+        </geometry>
+        <material name="">
+          <color rgba="1 1 0 1"/>
+        </material>
+      </visual>
+      <collision>
+        <origin rpy="0 0 0" xyz="0 0 0"/>
+        <geometry>
+          <mesh filename="file://$(find ar_description)/meshes/ar4/link_2.STL"/>
         </geometry>
       </collision>
@@ -101,14 +101,14 @@
         <origin rpy="0 0 0" xyz="0 0 0"/>
         <geometry>
-          <mesh filename="file://$(find ar_description)/meshes/${robot_parameters['mesh_dir']}/link_3.STL"/>
-        </geometry>
-        <material name="">
-          <color rgba="1 1 0 1"/>
-        </material>
-      </visual>
-      <collision>
-        <origin rpy="0 0 0" xyz="0 0 0"/>
-        <geometry>
-          <mesh filename="file://$(find ar_description)/meshes/${robot_parameters['mesh_dir']}/link_3.STL"/>
+          <mesh filename="file://$(find ar_description)/meshes/ar4/link_3.STL"/>
+        </geometry>
+        <material name="">
+          <color rgba="1 1 0 1"/>
+        </material>
+      </visual>
+      <collision>
+        <origin rpy="0 0 0" xyz="0 0 0"/>
+        <geometry>
+          <mesh filename="file://$(find ar_description)/meshes/ar4/link_3.STL"/>
         </geometry>
       </collision>
@@ -130,14 +130,14 @@
         <origin rpy="0 0 0" xyz="0 0 0"/>
         <geometry>
-          <mesh filename="file://$(find ar_description)/meshes/${robot_parameters['mesh_dir']}/link_4.STL"/>
-        </geometry>
-        <material name="">
-          <color rgba="1 1 0 1"/>
-        </material>
-      </visual>
-      <collision>
-        <origin rpy="0 0 0" xyz="0 0 0"/>
-        <geometry>
-          <mesh filename="file://$(find ar_description)/meshes/${robot_parameters['mesh_dir']}/link_4.STL"/>
+          <mesh filename="file://$(find ar_description)/meshes/ar4/link_4.STL"/>
+        </geometry>
+        <material name="">
+          <color rgba="1 1 0 1"/>
+        </material>
+      </visual>
+      <collision>
+        <origin rpy="0 0 0" xyz="0 0 0"/>
+        <geometry>
+          <mesh filename="file://$(find ar_description)/meshes/ar4/link_4.STL"/>
         </geometry>
       </collision>
@@ -159,14 +159,14 @@
         <origin rpy="0 0 0" xyz="0 0 0"/>
         <geometry>
-          <mesh filename="file://$(find ar_description)/meshes/${robot_parameters['mesh_dir']}/link_5.STL"/>
-        </geometry>
-        <material name="">
-          <color rgba="1 1 0 1"/>
-        </material>
-      </visual>
-      <collision>
-        <origin rpy="0 0 0" xyz="0 0 0"/>
-        <geometry>
-          <mesh filename="file://$(find ar_description)/meshes/${robot_parameters['mesh_dir']}/link_5.STL"/>
+          <mesh filename="file://$(find ar_description)/meshes/ar4/link_5.STL"/>
+        </geometry>
+        <material name="">
+          <color rgba="1 1 0 1"/>
+        </material>
+      </visual>
+      <collision>
+        <origin rpy="0 0 0" xyz="0 0 0"/>
+        <geometry>
+          <mesh filename="file://$(find ar_description)/meshes/ar4/link_5.STL"/>
         </geometry>
       </collision>
@@ -188,14 +188,14 @@
         <origin rpy="0 0 0" xyz="0 0 0"/>
         <geometry>
-          <mesh filename="file://$(find ar_description)/meshes/${robot_parameters['mesh_dir']}/link_6.STL"/>
-        </geometry>
-        <material name="">
-          <color rgba="1 1 0 1"/>
-        </material>
-      </visual>
-      <collision>
-        <origin rpy="0 0 0" xyz="0 0 0"/>
-        <geometry>
-          <mesh filename="file://$(find ar_description)/meshes/${robot_parameters['mesh_dir']}/link_6.STL"/>
+          <mesh filename="file://$(find ar_description)/meshes/ar4/link_6.STL"/>
+        </geometry>
+        <material name="">
+          <color rgba="1 1 0 1"/>
+        </material>
+      </visual>
+      <collision>
+        <origin rpy="0 0 0" xyz="0 0 0"/>
+        <geometry>
+          <mesh filename="file://$(find ar_description)/meshes/ar4/link_6.STL"/>
         </geometry>
       </collision>

File: src/ar_hardware_interface/urdf/ar.urdf.xacro (robot description, xacro)
@@ -4,5 +4,5 @@
   <xacro:arg name="arduino_serial_port" default="/dev/ttyUSB0"/>
   <xacro:arg name="calibrate" default="True"/>
-  <xacro:arg name="include_gripper" default="true"/>
+  <xacro:arg name="include_gripper" default="false"/>
   <xacro:include filename="$(find ar_description)/urdf/ar_macro.xacro"/>
   <xacro:include filename="$(find ar_description)/urdf/ar.ros2_control.xacro"/>
